Commit message: [FIXED] fix urdf

File: urdf/zed.urdf (robot description, URDF)
Before this commit: robot zed_camera, 4 links, 3 joints
Joints:
- joint zed_depth_camera_joint: origin xyz=0 0 0 rpy=-1.5707963267948966 0 -1.5707963267948966 -> xyz=0 0 0 rpy=0 0 0
- joint zed_left_camera_joint: origin xyz=0 0.06 0 rpy=0 0 0 -> xyz=0 0.06 0 rpy=-1.5707963267948966 0 -1.5707963267948966
- joint zed_right_camera_joint: origin xyz=0 -0.06 0 rpy=0 0 0 -> xyz=0 -0.06 0 rpy=-1.5707963267948966 0 -1.5707963267948966
